Commit message: feat(rl): Add IMU and contact sensors to URDF and create RL Inference node skeleton

File: src/mini_cheetah_demo/urdf/mini_cheetah.urdf.xacro (robot description, xacro)
@@ -53,4 +53,10 @@
   <gazebo reference="base_link">
     <material>Gazebo/DarkGrey</material>
+    <sensor name="imu_sensor" type="imu">
+      <always_on>1</always_on>
+      <update_rate>100</update_rate>
+      <visualize>true</visualize>
+      <topic>/imu</topic>
+    </sensor>
   </gazebo>
   <!-- ==================== 单腿 3 自由度 Xacro 宏 ==================== -->
@@ -168,5 +174,5 @@
         <material name="red"/>
       </visual>
-      <collision>
+      <collision name="${prefix}_foot_collision">
         <origin xyz="0 0 0" rpy="0 0 0"/>
         <geometry>
@@ -189,4 +195,13 @@
       <min_depth>0.001</min_depth>
       <material>Gazebo/Red</material>
+      <!-- 强化学习所需的接触力传感器 -->
+      <sensor name="${prefix}_contact_sensor" type="contact">
+        <always_on>true</always_on>
+        <update_rate>100</update_rate>
+        <contact>
+          <collision>${prefix}_foot_collision</collision>
+        </contact>
+        <topic>/contact/${prefix}</topic>
+      </sensor>
     </gazebo>
     <!-- Gazebo Harmonic 关节位置闭环 PID 力矩控制器 -->
@@ -244,4 +259,9 @@
       <odom_publish_frequency>50</odom_publish_frequency>
     </plugin>
+    <!-- RL 传感器系统插件 -->
+    <plugin filename="gz-sim-imu-system" name="gz::sim::systems::Imu">
+    </plugin>
+    <plugin filename="gz-sim-contact-system" name="gz::sim::systems::Contact">
+    </plugin>
   </gazebo>
 </robot>
